Commit message: speed up and tested

File: src/panda_ign_moveit2/panda_description/urdf/panda.urdf.xacro (robot description, xacro)
@@ -35,5 +35,5 @@
   <xacro:arg name="ros2_control_plugin" default="ign"/>
   <!-- The output control command interface provided by ros2_control ('position', 'velocity', 'effort' or certain combinations 'position,velocity') -->
-  <xacro:arg name="ros2_control_command_interface" default="effort"/>
+  <xacro:arg name="ros2_control_command_interface" default="position"/>
   <!-- The filepath to parameters of ROS 2 controllers -->
   <xacro:arg name="ros2_controller_parameters" default="$(find panda_moveit_config)/config/controllers_$(arg ros2_control_command_interface).yaml"/>

File: src/panda_ign_moveit2/panda_description/urdf/panda_utils.xacro (robot description, xacro)
@@ -163,10 +163,11 @@
   ">
     <link name="${link_name}">
-      <xacro:if value="${gazebo_preserve_fixed_joint}">
-        <inertial>
-          <mass value="1e-5"/>
-          <inertia ixx="1e-35" iyy="1e-35" izz="1e-35" ixy="0.0" ixz="0.0" iyz="0.0"/>
-        </inertial>
-      </xacro:if>
+      <xacro:unless value="${link_name == 'world'}">
+         <inertial>
+           <mass value="0.01"/>
+           <origin xyz="0 0 0" rpy="0 0 0"/>
+           <inertia ixx="0.001" ixy="0.0" ixz="0.0" iyy="0.001" iyz="0.0" izz="0.001"/>
+         </inertial>
+      </xacro:unless>
     </link>
     <!-- Preserve fixed joint, if desired -->
